Commit message: Add handrail to cargo bag

File: astrobee/description/description/urdf/model_cargo.urdf.xacro (robot description, xacro)
@@ -19,5 +19,5 @@
 <robot xmlns:xacro="http://www.ros.org/wiki/xacro">
   <gazebo>
-    <plugin name="cargo_ros" filename="libgazebo_model_plugin_cargo.so">>
+    <plugin name="cargo_ros" filename="libgazebo_model_plugin_cargo.so">
       <namespace>/${ns}/</namespace>
       <rate>10.0</rate>          <!-- Rate at which dock state checked  -->

File: description/urdf/cargo_bag.urdf.xacro (robot description, xacro)
@@ -2,10 +2,10 @@
 <robot name="cargo" xmlns:xacro="http://www.ros.org/wiki/xacro">
   <link name="body">
-<!--     <collision>
+    <collision>
       <origin xyz="0 0 0" rpy="0 0 0" />
       <geometry>
         <mesh filename="package://isaac_description/meshes/half_ctb_02_4.dae" scale="1 1 1"/>
       </geometry>
-    </collision> -->
+    </collision>
     <visual>
       <origin xyz="0 0 0" rpy="0 0 0" />
@@ -26,8 +26,20 @@
       </geometry>
     </visual>
+    <collision>
+      <origin xyz="0.1 -0.21 0" rpy="0 0 -1.57" />
+      <geometry>
+        <mesh filename="package://astrobee_handrail_8_5/meshes/handrail_8_5.dae"/>
+      </geometry>
+    </collision>
+    <visual>
+      <origin xyz="0.1 -0.21 0" rpy="0 0 -1.57" />
+      <geometry>
+        <mesh filename="package://astrobee_handrail_8_5/meshes/handrail_8_5.dae"/>
+      </geometry>
+    </visual>
     <inertial>
-      <mass value="0.5" />
+      <mass value="9.58" />
       <origin xyz="0 0 0" rpy="0 0 0" />
-      <inertia ixx="1" ixy="0" ixz="0" iyy="1" iyz="0" izz="1" />
+      <inertia ixx="0.153427995" ixy="0" ixz="0" iyy="0.14271405" iyz="0" izz="0.162302759" />
     </inertial>
   </link>
